Commit message: Update urdf_from_xacro.urdf

File: navvis_description/urdf/urdf_from_xacro.urdf (robot description, URDF)
Before this commit: robot robot, 7 links, 6 joints
Links:
- added link laser_horiz_base_link, mass 0.83; collision cylinder length=0.0717 radius=0.0516; visual mesh filename=package://velodyne_description/meshes/VLP16_base_1.dae
- added link wheel_center; collision cylinder length=0.05 radius=0.15; visual cylinder length=0.05 radius=0.15
- link laser_horiz: mass None -> 0.01; geometry collision sphere radius=0; visual mesh filename=package://velodyne_description/meshes/VLP16_scan.dae
- link laser_vert_bottom: mass None -> 1e-5; geometry collision box size=0.1 0.1 0.1; visual mesh filename=package://gazebo_plugins/test/multi_robot_scenario/meshes/l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
- link laser_vert_top_left: mass None -> 1e-5; geometry collision box size=0.1 0.1 0.1; visual mesh filename=package://gazebo_plugins/test/multi_robot_scenario/meshes/l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
- link laser_vert_top_right: mass None -> 1e-5; geometry collision box size=0.1 0.1 0.1; visual mesh filename=package://gazebo_plugins/test/multi_robot_scenario/meshes/l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
Joints:
- removed joint base_laser_horiz_joint
- added joint base_wheel_center_joint: type continuous, parent base, child wheel_center, origin xyz=0.10 0.0 0.0 rpy=-1.57079632679 0.0 0.0, axis 0.0 0.0 1.0, limit effort=1000.0 velocity=80.0
- added joint laser_horiz_base_mount_joint: type fixed, parent base, child laser_horiz_base_link, origin xyz=0.2325416305773505 -0.0001380069427607134 1.920122926231907 rpy=-0.0012068 0.114646 -0.0015308
- added joint laser_horiz_base_scan_joint: type fixed, parent laser_horiz_base_link, child laser_horiz, origin xyz=0 0 0.0377 rpy=0 0 0
- joint base_laser_vert_bottom_joint: axis (none) -> 0 0 1; origin xyz=0.3158 -0.0021 0.5100 rpy=3.1355 -1.3045 0.0025 -> xyz=0.3157894464801903 -0.002068548615034871 0.5099999434059285 rpy=3.1354753 -1.3045001 0.0024658
- joint base_laser_vert_top_left_joint: axis (none) -> 0 0 1
- joint base_laser_vert_top_right_joint: axis (none) -> 0 0 1
- joint base_wheel_left_joint: axis (none) -> 0.0 0.0 1.0; limit (none) -> effort=1000.0 velocity=80.0; type fixed -> continuous
- joint base_wheel_right_joint: axis (none) -> 0.0 0.0 1.0; limit (none) -> effort=1000.0 velocity=80.0; type fixed -> continuous
